Commit message: los meros launch

File: robotino/catkin_ws/src/robotino_description/robotino_tesis.urdf (robot description, URDF)
Before this commit: robot robotino, 7 links, 6 joints
Links:
- removed link kinect_link
- added link depth_device_link; visual box size=0.03 0.14 0.0175
Joints:
- joint base_to_kinect: child kinect_link -> depth_device_link

Commit message: aruco_mapping ok

File: robotino/catkin_ws/src/robotino_description/robotino_tesis.urdf (robot description, URDF)
Before this commit: robot robotino, 7 links, 6 joints
Links:
- removed link depth_device_link
- added link zed_link; visual box size=0.03 0.14 0.0175
Joints:
- joint base_to_kinect: child depth_device_link -> zed_link
